File: boat_pcb_v2/com_board/com_board.kicad_sch (KiCad schematic)
At the start: 62 parts, among them J1 Conn_01x26_Socket, J2 USB_C_Receptacle_USB2.0_16P, J5 Conn_01x26_Socket, J7 XBP9B-DMUTB002, J8 Conn_01x02_Pin, J9 Conn_01x26_Socket, Q1 NMOS, U1 Particle_B404X, U2 AP62301WU-7, U3 AP62301WU-7

Commit message: Changed folders for symbols and footprints
Parts:
- D2, D4: footprint Com_Board_Parts_Lib:SMB -> WaterNet26_Parts_Lib:SMB
- D3: footprint Com_Board_Parts_Lib:LED_CLMVC-FKA-CL1D1L71BB7C3C3 -> WaterNet26_Parts_Lib:LED_CLMVC-FKA-CL1D1L71BB7C3C3
- J7: footprint Com_Board_Parts_Lib:SULLINS_NPPN101BFCN-RC -> WaterNet26_Parts_Lib:SULLINS_NPPN101BFCN-RC
- JP2, JP3: footprint Com_Board_Parts_Lib:B04B-PASK-1 -> WaterNet26_Parts_Lib:B04B-PASK-1
- L1, L2, L3: footprint Com_Board_Parts_Lib:INDC1608X95N -> WaterNet26_Parts_Lib:INDC1608X95N
- Q1: footprint Com_Board_Parts_Lib:SOT95P240X110-3N -> WaterNet26_Parts_Lib:SOT95P240X110-3N
- U1: footprint Com_Board_Parts_Lib:b404x -> WaterNet26_Parts_Lib:b404x
- U2, U3: footprint Com_Board_Parts_Lib:SOT95P280X100-6N -> WaterNet26_Parts_Lib:SOT95P280X100-6N
Changed lines of the file:
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@@
 			)
 		)
-		(property "Footprint" "Com_Board_Parts_Lib:INDC1608X95N"
+		(property "Footprint" "WaterNet26_Parts_Lib:INDC1608X95N"
 			(at 86.36 26.67 0)
 			(effects
@@
 			)
 		)
-		(property "Footprint" "Com_Board_Parts_Lib:SULLINS_NPPN101BFCN-RC"
+		(property "Footprint" "WaterNet26_Parts_Lib:SULLINS_NPPN101BFCN-RC"
 			(at 308.61 151.13 0)
 			(effects
@@
 			)
 		)
-		(property "Footprint" "Com_Board_Parts_Lib:SMB"
+		(property "Footprint" "WaterNet26_Parts_Lib:SMB"
 			(at 323.85 200.66 0)
 			(effects
@@
 			)
 		)
-		(property "Footprint" "Com_Board_Parts_Lib:SOT95P280X100-6N"
+		(property "Footprint" "WaterNet26_Parts_Lib:SOT95P280X100-6N"
 			(at 265.43 97.79 0)
 			(effects
@@
 			)
 		)
-		(property "Footprint" "Com_Board_Parts_Lib:SOT95P280X100-6N"
+		(property "Footprint" "WaterNet26_Parts_Lib:SOT95P280X100-6N"
 			(at 264.16 38.1 0)
 			(effects
@@
 			)
 		)
-		(property "Footprint" "Com_Board_Parts_Lib:B04B-PASK-1"
+		(property "Footprint" "WaterNet26_Parts_Lib:B04B-PASK-1"
 			(at 166.37 231.14 0)
 			(effects
@@
 			)
 		)
-		(property "Footprint" "Com_Board_Parts_Lib:LED_CLMVC-FKA-CL1D1L71BB7C3C3"
+		(property "Footprint" "WaterNet26_Parts_Lib:LED_CLMVC-FKA-CL1D1L71BB7C3C3"
 			(at 242.57 228.6 0)
 			(effects
@@
 			)
 		)
-		(property "Footprint" "Com_Board_Parts_Lib:B04B-PASK-1"
+		(property "Footprint" "WaterNet26_Parts_Lib:B04B-PASK-1"
 			(at 130.81 231.14 0)
 			(effects
@@
 			)
 		)
-		(property "Footprint" "Com_Board_Parts_Lib:b404x"
+		(property "Footprint" "WaterNet26_Parts_Lib:b404x"
 			(at 135.89 21.59 0)
 			(effects
@@
 			)
 		)
-		(property "Footprint" "Com_Board_Parts_Lib:INDC1608X95N"
+		(property "Footprint" "WaterNet26_Parts_Lib:INDC1608X95N"
 			(at 299.72 33.02 0)
 			(effects
@@
 			)
 		)
-		(property "Footprint" "Com_Board_Parts_Lib:SMB"
+		(property "Footprint" "WaterNet26_Parts_Lib:SMB"
 			(at 323.85 209.55 0)
 			(effects
@@
 			)
 		)
-		(property "Footprint" "Com_Board_Parts_Lib:INDC1608X95N"
+		(property "Footprint" "WaterNet26_Parts_Lib:INDC1608X95N"
 			(at 300.99 92.71 0)
 			(effects
@@
 			)
 		)
-		(property "Footprint" "Com_Board_Parts_Lib:SOT95P240X110-3N"
+		(property "Footprint" "WaterNet26_Parts_Lib:SOT95P240X110-3N"
 			(at 148.59 165.1 0)
 			(effects
