File: boat_pcb_v2/WN_com_board/com_board.kicad_pcb (KiCad board)
At the start: 2 copper layers, 9 parts, among them J2 USB_C_Receptacle_USB2.0_16P, J7 XBP9B-DMUTB002, U1 Particle_B404X, U2 AP62301WU-7, U3 AP62301WU-7

Commit message: Updated submodule
Parts:
- added C1: 1µ, 25V, Capacitor_SMD:C_0603_1608Metric_Pad1.08x0.95mm_HandSolder, F.Cu at (84.1, 61.3)
- added C10: 10µ, 25V, Capacitor_SMD:C_0603_1608Metric_Pad1.08x0.95mm_HandSolder, F.Cu at (88.4, 61.3)
- added C11: 0.1µ, 25V, Capacitor_SMD:C_0603_1608Metric_Pad1.08x0.95mm_HandSolder, F.Cu at (88.4, 63.8)
- added C12: 0.1µ, 25V, Capacitor_SMD:C_0603_1608Metric_Pad1.08x0.95mm_HandSolder, F.Cu at (88.4, 66.3)
- added C13: 10µ, 25V, Capacitor_SMD:C_0603_1608Metric_Pad1.08x0.95mm_HandSolder, F.Cu at (88.4, 68.8)
- added C14: 47µ, 6.3V, Capacitor_SMD:C_0603_1608Metric_Pad1.08x0.95mm_HandSolder, F.Cu at (88.4, 71.4)
- added C15: 10µ, 25V, Capacitor_SMD:C_0603_1608Metric_Pad1.08x0.95mm_HandSolder, F.Cu at (88.4, 73.9)
- added C16: 0.1µ, 25V, Capacitor_SMD:C_0603_1608Metric_Pad1.08x0.95mm_HandSolder, F.Cu at (88.4, 76.4)
- added C17: 0.1µ, 25V, Capacitor_SMD:C_0603_1608Metric_Pad1.08x0.95mm_HandSolder, F.Cu at (88.4, 78.9)
- added C2: 1µ, 25V, Capacitor_SMD:C_0603_1608Metric_Pad1.08x0.95mm_HandSolder, F.Cu at (84.1, 63.8)
- added C20: 1µ, 25V, Capacitor_SMD:C_0603_1608Metric_Pad1.08x0.95mm_HandSolder, F.Cu at (92.8, 61.3)
- added C21: 1µ, 25V, Capacitor_SMD:C_0603_1608Metric_Pad1.08x0.95mm_HandSolder, F.Cu at (92.8, 63.8)
- added C22: 0.1µ, 25V, Capacitor_SMD:C_0603_1608Metric_Pad1.08x0.95mm_HandSolder, F.Cu at (92.8, 66.3)
- added C23: 10µ, 25V, Capacitor_SMD:C_0603_1608Metric_Pad1.08x0.95mm_HandSolder, F.Cu at (92.8, 68.8)
- added C24: 10µ, 25V, Capacitor_SMD:C_0603_1608Metric_Pad1.08x0.95mm_HandSolder, F.Cu at (92.8, 71.4)
- added C25: 0.1µ, 25V, Capacitor_SMD:C_0603_1608Metric_Pad1.08x0.95mm_HandSolder, F.Cu at (92.8, 73.9)
- added C26: 1µ, 25V, Capacitor_SMD:C_0603_1608Metric_Pad1.08x0.95mm_HandSolder, F.Cu at (92.8, 76.4)
- added C3: 1µ, 25V, Capacitor_SMD:C_0603_1608Metric_Pad1.08x0.95mm_HandSolder, F.Cu at (84.1, 66.3)
- added C4: 1µ, 25V, Capacitor_SMD:C_0603_1608Metric_Pad1.08x0.95mm_HandSolder, F.Cu at (84.1, 68.8)
- added C5: 0.1µ, 25V, Capacitor_SMD:C_0603_1608Metric_Pad1.08x0.95mm_HandSolder, F.Cu at (84.1, 71.4)
- added C7: 0.1µ, 25V, Capacitor_SMD:C_0603_1608Metric_Pad1.08x0.95mm_HandSolder, F.Cu at (84.1, 73.9)
- added C8: 10µ, 25V, Capacitor_SMD:C_0603_1608Metric_Pad1.08x0.95mm_HandSolder, F.Cu at (84.1, 76.4)
- added C9: 47µ, 6.3V, Capacitor_SMD:C_0603_1608Metric_Pad1.08x0.95mm_HandSolder, F.Cu at (84.1, 78.9)
- added D2: D_Schottky, WN_com_board:SMB, F.Cu at (113.6, 119.3)
- added D4: D_Schottky, WN_com_board:SMB, F.Cu at (113.6, 124.2)
- added J1: Conn_01x26_Socket, Connector_PinHeader_2.54mm:PinHeader_1x26_P2.54mm_Vertical, F.Cu at (70.4, 62.4)
- added J5: Conn_01x26_Socket, Connector_PinHeader_2.54mm:PinHeader_1x26_P2.54mm_Vertical, F.Cu at (75.0, 62.4)
- added J8: Conn_01x02_Pin, Connector_PinHeader_2.54mm:PinHeader_1x02_P2.54mm_Vertical, F.Cu at (84.2, 100.0)
- added J9: Conn_01x26_Socket, Connector_PinHeader_2.54mm:PinHeader_1x26_P2.54mm_Vertical, F.Cu at (79.6, 62.4)
- added L1: 3.3µ, WN_com_board:INDC1608X95N, F.Cu at (111.7, 128.0)
- added L2: 3.3µ, WN_com_board:INDC1608X95N, F.Cu at (111.7, 130.5)
- added L3: 3.3µ, WN_com_board:INDC1608X95N, F.Cu at (111.7, 133.0)
- added Q1: NMOS, WN_com_board:SOT95P240X110-3N, F.Cu at (98.6, 134.1)
- added R10: 37.4k, Resistor_SMD:R_0603_1608Metric, F.Cu at (87.9, 81.4)
- added R11: 10k, Resistor_SMD:R_0603_1608Metric, F.Cu at (87.9, 83.9)
- added R12: 50k, Resistor_SMD:R_0603_1608Metric, F.Cu at (87.9, 86.4)
- added R13: 50k, Resistor_SMD:R_0603_1608Metric, F.Cu at (87.9, 88.9)
- added R14: 2.2k, Resistor_SMD:R_0603_1608Metric, F.Cu at (87.9, 91.4)
- added R15: 2.2k, Resistor_SMD:R_0603_1608Metric, F.Cu at (87.9, 94.0)
- added R16: 0R, Resistor_SMD:R_0603_1608Metric, F.Cu at (87.9, 96.5)
- added R17: 330, Resistor_SMD:R_0603_1608Metric, F.Cu at (91.9, 81.4)
- added R18: 330, Resistor_SMD:R_0603_1608Metric, F.Cu at (91.9, 83.9)
- added R19: 330, Resistor_SMD:R_0603_1608Metric, F.Cu at (91.9, 86.4)
- added R2: 5.1k, Resistor_SMD:R_0603_1608Metric, F.Cu at (83.9, 81.4)
- added R20: 100k, Resistor_SMD:R_0603_1608Metric, F.Cu at (91.9, 88.9)
- added R3: 5.1k, Resistor_SMD:R_0603_1608Metric, F.Cu at (83.9, 83.9)
- added R4: 100k, Resistor_SMD:R_0603_1608Metric, F.Cu at (83.9, 86.4)
- added R6: 100k, Resistor_SMD:R_0603_1608Metric, F.Cu at (83.9, 88.9)
- added R7: 31.6k, Resistor_SMD:R_0603_1608Metric, F.Cu at (83.9, 91.4)
- added R8: 10k, Resistor_SMD:R_0603_1608Metric, F.Cu at (83.9, 94.0)
- added R9: 100k, Resistor_SMD:R_0603_1608Metric, F.Cu at (83.9, 96.5)
- added S1: TS04-66-50-BK-160-SMT-TR, WN_com_board:SW_TS04-66-50-BK-160-SMT-TR, F.Cu at (103.3, 120.7)
- added S2: TS04-66-50-BK-160-SMT-TR, WN_com_board:SW_TS04-66-50-BK-160-SMT-TR, F.Cu at (103.3, 128.2)
- D3: footprint Com_Board_Parts_Lib:LED_CLMVC-FKA-CL1D1L71BB7C3C3 -> WN_com_board:LED_CLMVC-FKA-CL1D1L71BB7C3C3
- J7: footprint Com_Board_Parts_Lib:SULLINS_NPPN101BFCN-RC -> WN_com_board:SULLINS_NPPN101BFCN-RC
- JP2, JP3: footprint Com_Board_Parts_Lib:B04B-PASK-1 -> WN_com_board:B04B-PASK-1
- U1: footprint Com_Board_Parts_Lib:b404x -> WN_com_board:b404x
- U2, U3: footprint Com_Board_Parts_Lib:SOT95P280X100-6N -> WN_com_board:SOT95P280X100-6N
