File: boat_pcb_v2/WN_com_board/com_board.kicad_sch (KiCad schematic)
At the start: 62 parts, among them J1 Conn_01x26_Socket, J2 USB_C_Receptacle_USB2.0_16P, J5 Conn_01x26_Socket, J7 XBP9B-DMUTB002, J8 Conn_01x02_Pin, J9 Conn_01x26_Socket, Q1 NMOS, U1 Particle_B404X, U2 AP62301WU-7, U3 AP62301WU-7

Commit message: Updated submodule
Parts:
- C1, C10, C11, C12, C13, C14, C15, C16, C17, C2, C20, C21, C22, C23, C24, C25, C26, C3, C4, C5, C7, C8, C9: symbol Device:C -> WN_com_board:C
- D1: symbol Power_Protection:USBLC6-2SC6 -> WN_com_board:USBLC6-2SC6
- D2, D4: footprint WaterNet26_Parts_Lib:SMB -> WN_com_board:SMB; symbol Device:D_Schottky -> WN_com_board:D_Schottky
- D3: footprint WaterNet26_Parts_Lib:LED_CLMVC-FKA-CL1D1L71BB7C3C3 -> WN_com_board:LED_CLMVC-FKA-CL1D1L71BB7C3C3; symbol on_board_led:CLMVC-FKA-CL1D1L71BB7C3C3 -> WN_com_board:CLMVC-FKA-CL1D1L71BB7C3C3
- J1, J5, J9: symbol Connector:Conn_01x26_Socket -> WN_com_board:Conn_01x26_Socket
- J2: symbol Connector:USB_C_Receptacle_USB2.0_16P -> WN_com_board:USB_C_Receptacle_USB2.0_16P
- J7: footprint WaterNet26_Parts_Lib:SULLINS_NPPN101BFCN-RC -> WN_com_board:SULLINS_NPPN101BFCN-RC; symbol com_board_library:XBP9B-DMUTB002 -> WN_com_board:XBP9B-DMUTB002
- J8: symbol Connector:Conn_01x02_Pin -> WN_com_board:Conn_01x02_Pin
- JP2, JP3: footprint WaterNet26_Parts_Lib:B04B-PASK-1 -> WN_com_board:B04B-PASK-1; symbol com_board_library:B04B-PASK-1 -> WN_com_board:B04B-PASK-1_1
- L1, L2, L3: footprint WaterNet26_Parts_Lib:INDC1608X95N -> WN_com_board:INDC1608X95N; symbol Device:L -> WN_com_board:L
- Q1: footprint WaterNet26_Parts_Lib:SOT95P240X110-3N -> WN_com_board:SOT95P240X110-3N; symbol Simulation_SPICE:NMOS -> WN_com_board:NMOS
- R10, R11, R12, R13, R14, R15, R16, R17, R18, R19, R2, R20, R3, R4, R6, R7, R8, R9: symbol Device:R -> WN_com_board:R
- S1, S2: footprint TS04-66-50-BK-160-SMT-TR:SW_TS04-66-50-BK-160-SMT-TR -> WN_com_board:SW_TS04-66-50-BK-160-SMT-TR; symbol push_button:TS04-66-50-BK-160-SMT-TR -> WN_com_board:TS04-66-50-BK-160-SMT-TR
- U1: footprint WaterNet26_Parts_Lib:b404x -> WN_com_board:b404x; symbol com_board_library:Particle_B404X -> WN_com_board:Particle_B404X
- U2, U3: footprint WaterNet26_Parts_Lib:SOT95P280X100-6N -> WN_com_board:SOT95P280X100-6N; symbol Regulators:AP62301WU-7 -> WN_com_board:AP62301WU-7

Commit message: Changes made to footprints and symbols in existing schematics
Parts:
- removed C3, C4: 1µ, 25V, Capacitor_SMD:C_0603_1608Metric_Pad1.08x0.95mm_HandSolder, symbol WN_com_board:C
- removed D1: USBLC6-2SC6, Package_TO_SOT_SMD:SOT-23-6, symbol WN_com_board:USBLC6-2SC6
- removed D3: CLMVC-FKA-CL1D1L71BB7C3C3, WN_com_board:LED_CLMVC-FKA-CL1D1L71BB7C3C3, symbol WN_com_board:CLMVC-FKA-CL1D1L71BB7C3C3
- removed J2: USB_C_Receptacle_USB2.0_16P, Connector_USB:USB_C_Plug_ShenzhenJingTuoJin_918-118A2021Y40002_Vertical, symbol WN_com_board:USB_C_Receptacle_USB2.0_16P
- removed L3: 3.3µ, WN_com_board:INDC1608X95N, symbol WN_com_board:L
- removed R16: 0R, Resistor_SMD:R_0603_1608Metric, symbol WN_com_board:R
- removed R17, R18, R19: 330, Resistor_SMD:R_0603_1608Metric, symbol WN_com_board:R
- removed R2, R3: 5.1k, Resistor_SMD:R_0603_1608Metric, symbol WN_com_board:R
- removed U1: Particle_B404X, WN_com_board:b404x, symbol WN_com_board:Particle_B404X
- added C27, C28: 1µ, 100V, WaterNet26 Footprints:CAPC2012X145N, symbol Device:C
- added C68, C69, C76: 0.1uF 25V, WaterNet26 Footprints:CAPC2012X95N, symbol WaterNet26 Library:CL21B104KACNNNC
- added D11: CLMVC-FKA-CL1D1L71BB7C3C3, WaterNet26 Footprints:LED_CLMVC-FKA-CL1D1L71BB7C3C3, symbol WaterNet26 Library:CLMVC-FKA-CL1D1L71BB7C3C3
- added D5: USBLC6-2SC6, Package_TO_SOT_SMD:SOT-23-6, symbol Power_Protection:USBLC6-2SC6
- added J16: USB4120-03-C_REVA6, WaterNet26 Footprints:GCT_USB4120-03-C_REVA6, symbol WaterNet26 Library:USB4120-03-C_REVA6
- added L6: 3.3µ, WaterNet26 Footprints:INDC1608X95N, symbol Device:L
- added R25, R26: 5.1K, WaterNet26 Footprints:RESC1508X55N, symbol WaterNet26 Library:RMCF0603FT5K10
- added R31, R32, R33: 100 Ohm, WaterNet26 Footprints:RES_ERJ3EKF1000V, symbol WaterNet26 Library:ERJ3EKF1000V
- added R66, R67, R68: 10K, WaterNet26 Footprints:RES_ERA6AEB103V, symbol WaterNet26 Library:ERA6AEB103V
- added U1: Particle_B404X, WaterNet26 Footprints:b404x, symbol WaterNet26 Library:Particle_B404X
- added U16, U17, U18: BSS123-7-F, WaterNet26 Footprints:SOT95P240X110-3N, symbol WaterNet26 Library:BSS123-7-F
- C1, C2, C20, C21, C26: value 1µ, 25V -> 1µ, 100V; footprint Capacitor_SMD:C_0603_1608Metric_Pad1.08x0.95mm_HandSolder -> WaterNet26 Footprints:CAPC2012X145N; symbol WN_com_board:C -> Device:C
- C10, C13, C15, C23, C24, C8: footprint Capacitor_SMD:C_0603_1608Metric_Pad1.08x0.95mm_HandSolder -> WaterNet26 Footprints:CAPC2012X145N; symbol WN_com_board:C -> Device:C
- C11, C12, C16, C17, C22, C25, C5, C7: footprint Capacitor_SMD:C_0603_1608Metric_Pad1.08x0.95mm_HandSolder -> WaterNet26 Footprints:CAPC2012X95N; symbol WN_com_board:C -> Device:C
- C14, C9: footprint Capacitor_SMD:C_0603_1608Metric_Pad1.08x0.95mm_HandSolder -> WaterNet26 Footprints:CAPC3216X180N; symbol WN_com_board:C -> Device:C
- D2, D4: value D_Schottky -> RB070MM-30TR; footprint WN_com_board:SMB -> WaterNet26 Footprints:DIO_RB070MM-30TR; symbol WN_com_board:D_Schottky -> WaterNet26 Library:RB070MM-30TR
- J1, J5, J9: symbol WN_com_board:Conn_01x26_Socket -> Connector:Conn_01x26_Socket
- J7: footprint WN_com_board:SULLINS_NPPN101BFCN-RC -> WaterNet26 Footprints:SULLINS_NPPN101BFCN-RC; symbol WN_com_board:XBP9B-DMUTB002 -> WaterNet26 Library:XBP9B-DMUTB002
- J8: symbol WN_com_board:Conn_01x02_Pin -> Connector:Conn_01x02_Pin
- JP2, JP3: footprint WN_com_board:B04B-PASK-1 -> WaterNet26 Footprints:B04B-PASK-1; symbol WN_com_board:B04B-PASK-1_1 -> WaterNet26 Library:B04B-PASK-1_1
- L1, L2: footprint WN_com_board:INDC1608X95N -> WaterNet26 Footprints:INDC1608X95N; symbol WN_com_board:L -> Device:L
- Q1: footprint WN_com_board:SOT95P240X110-3N -> WaterNet26 Footprints:SOT95P240X110-3N; symbol WN_com_board:NMOS -> Simulation_SPICE:NMOS
- R10: footprint Resistor_SMD:R_0603_1608Metric -> WaterNet26 Footprints:RESC1608X55N; symbol WN_com_board:R -> Device:R; MP RR0816P-3742-D-56C -> RT0603BRE0737K4L
- R11, R8: footprint Resistor_SMD:R_0603_1608Metric -> WaterNet26 Footprints:RES_ERA6AEB103V; symbol WN_com_board:R -> Device:R
- R12, R13, R14, R15: footprint Resistor_SMD:R_0603_1608Metric -> WaterNet26 Footprints:RESC1608X55N; symbol WN_com_board:R -> Device:R
- R20, R4, R6, R9: footprint Resistor_SMD:R_0603_1608Metric -> WaterNet26 Footprints:RES_ERA6AEB104V; symbol WN_com_board:R -> Device:R
- R7: footprint Resistor_SMD:R_0603_1608Metric -> WaterNet26 Footprints:RES_ERA6AEB3162V; symbol WN_com_board:R -> Device:R
- S1, S2: footprint WN_com_board:SW_TS04-66-50-BK-160-SMT-TR -> WaterNet26 Footprints:SW_TS04-66-50-BK-160-SMT-TR; symbol WN_com_board:TS04-66-50-BK-160-SMT-TR -> WaterNet26 Library:TS04-66-50-BK-160-SMT-TR
- U2, U3: footprint WN_com_board:SOT95P280X100-6N -> WaterNet26 Footprints:SOT95P280X100-6N; symbol WN_com_board:AP62301WU-7 -> WaterNet26 Library:AP62301WU-7
Connections:
- net +3V3: now also D11.1, U1.10 (3V3), U1.12 (3V3)
- net +3V8: now also U1.2 (VCC), U1.4 (VCC), U1.6 (VCC), U1.8 (VCC)
- net +VBUSF: now also D2.1, C28.1, L6.2, U1.16 (VUSB); no longer D2.2 (A)
- net A0: now also U1.23 (A0)
- net A1: now also U1.33 (A1)
- net A2: now also U1.35 (A2)
- net A3: now also U1.37 (A3)
- net A4: now also U1.41 (A4)
- net A5: now also U1.43 (A5)
- net A6: now also U1.45 (A6)
- net A7: now also U1.47 (A7)
- net BAT_12_IN: now also D4.1; no longer D4.2 (A)
- net CS: now also U1.48 (CS)
- net D2: now also U1.42 (D2)
- net D3: now also U1.40 (D3)
- net GND: now also C27.2, C28.2, C68.2, C69.2, C76.2, D5.2 (GND), J16.A1 (GND_A), J16.A12 (GND_A), J16.B1 (GND_B), J16.B12 (GND_B), J16.S1 (SHIELD), J16.S2 (SHIELD), J16.S3 (SHIELD), J16.S4 (SHIELD), R25.1, R26.1, R66.1, R67.1, R68.1, U1.1 (GND), U1.15 (GND), U1.21 (GND), U1.3 (GND), U1.39 (AGND), U1.49 (AGND), U1.5 (GND), U1.56 (GND), U1.7 (GND), U1.9 (GND), U1.S1 (SHIELD), U1.S2 (SHIELD), U16.2 (S), U17.2 (S), U18.2 (S)
- net GPIO0: now also U1.62 (GPIO0)
- net GPIO1: now also U1.64 (GPIO1)
- net MISO: now also U1.50 (MISO)
- net MODE: now also U1.32 (MODE); no longer C5.1, R4.2, S1.1, S1.3
- net MOSI: now also U1.52 (MOSI)
- net PWM0: now also U1.66 (PWM0)
- net PWM1: now also U1.68 (PWM1)
- net PWM2: now also U1.70 (PWM2)
- net PWM3: now also U1.72 (PWM3)
- net RESET: now also C5.1, R4.2, S1.1, S1.3, U1.34 (RESET)
- net RX: now also U1.38 (RX)
- net SCK: now also U1.54 (SCK)
- net SCL: now also U1.20 (SCL)
- net SDA: now also U1.22 (SDA)
- net TX: now also U1.36 (TX)
- net USB_D+_S: now also D5.4 (I/O2), U1.11 (USB_D+)
- net USB_D-_S: now also D5.6 (I/O1), U1.13 (USB_D-)
- net VSEL: now also D2.2, D4.2; no longer D2.1 (K), D4.1 (K)
- new net: R31.1, U16.3 (D)
- new net: D5.1 (I/O1), J16.A7 (D1-), J16.B7 (D2-)
- new net: D5.3 (I/O2), J16.A6 (D1+), J16.B6 (D2+)
- new net: R33.1, U18.3 (D)
- new net: J16.A5 (CC1), R25.2
- new net: J16.B5 (CC2), R26.2
- new net: D11.4, R33.2
- new net: D11.2, R31.2
- new net: R32.1, U17.3 (D)
- new net: D11.3, R32.2
- new net RGB_B: C68.1, R67.2, U1.65 (RGBB), U16.1 (G)
- new net RGB_G: C69.1, R66.2, U1.63 (RGBG), U17.1 (G)
- new net RGB_R: C76.1, R68.2, U1.61 (RGBR), U18.1 (G)
- new net VBUS_A: C27.1, D5.5 (VBUS), J16.A4 (VBUS_A), J16.A9 (VBUS_A), J16.B4 (VBUS_B), J16.B9 (VBUS_B), L6.1
Other:
- note added: "Onboard RGB LED"
- note removed: "On-board LEDs"
- moved on the sheet: C1, C10, C11, C12, C13, C14, C15, C16, C17, C2, C20, C21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
