File: boat_pcb_v2/WN_power_board/WaterNetPowerBoard.kicad_sch (KiCad schematic)
At the start: 204 parts, among them J1 USB4120-03-C_REVA6, J10 XT60-M, J13 XT60-F, J15 XT60-M, J16 TSW-108-07-F-D, J17 TSW-108-07-F-D, J18 TSW-108-07-F-D, J19 TSW-108-07-F-D, J2 USB4120-03-C_REVA6, J20 TSW-108-07-F-D, J21 TSW-108-07-F-D, J3 4 Pin Fan Header, J4 350761-4, J5 B2B-PH-K-S, J6 XT60-F, J7 XT60-M, J8 QWIIC, J9 QWIIC, Q1 SI7149ADP-T1-GE3, Q3 SI7149ADP-T1-GE3, SW2 Push Button, SW3 Push Button, U1 INA4181A3IPWR, U10 TPS922051D1DSGR, U11 TPS922051D1DSGR, U12 BSS123-7-F, U13 BSS123-7-F, U14 BSS123-7-F, U15 TMP117xxDRV, U16 BSS123-7-F, U17 BSS123-7-F, U18 BSS123-7-F, U2 MIC28514T-E_PHA, U3 MCP2200-I_SO, U4 BSS123-7-F, U5 BSS123-7-F, U6 AP62301WU-7, U7 BSS123-7-F, U8 ESP32-S3-WROOM-1, U9 TPS922051D1DSGR, Y1 ECS-120-12-33-AGN-TR

Commit message: Update WaterNetPowerBoard to reference fixed library submodule
Parts:
- C1, C14, C19, C25, C28, C32: footprint CL21B104KCFSFNE:CAPC2012X135N -> WaterNet26 Library:CAPC2012X135N; symbol WaterNetPowerBoardLibrary:CL21B104KCFSFNE -> WaterNet26 Library:CL21B104KCFSFNE
- C10, C13, C22, C3, C30, C35, C39, C45, C54, C8: footprint CL21A106KAYNNNE:CAPC2012X145N -> WaterNet26 Library:CAPC2012X145N; symbol WaterNetPowerBoardLibrary:CL21A106KAYNNNE -> WaterNet26 Library:CL21A106KAYNNNE
- C11, C12, C15, C16, C17, C18, C23, C24, C29, C33, C38, C4, C40, C41, C42, C46, C5, C53, C68, C69, C7, C70, C71, C74, C75, C76, C9: footprint CL21B104KACNNNC:CAPC2012X95N -> WaterNet26 Library:CAPC2012X95N; symbol WaterNetPowerBoardLibrary:CL21B104KACNNNC -> WaterNet26 Library:CL21B104KACNNNC
- C2, C26, C27, C31: footprint CL32Y106KCVZNWE:CAPC3225X280N -> WaterNet26 Library:CAPC3225X280N; symbol WaterNetPowerBoardLibrary:CL32Y106KCVZNWE -> WaterNet26 Library:CL32Y106KCVZNWE
- C20, C34, C43: footprint CL10B103KB8NNNC:CAPC1608X90N -> WaterNet26 Library:CAPC1608X90N; symbol WaterNetPowerBoardLibrary:CL10B103KB8NNNC -> WaterNet26 Library:CL10B103KB8NNNC
- C21, C44: footprint C3216X5R1E476M160AC:CAPC3216X180N -> WaterNet26 Library:CAPC3216X180N; symbol WaterNetPowerBoardLibrary:C3216X5R1E476M160AC -> WaterNet26 Library:C3216X5R1E476M160AC
- C36, C37: footprint CL10C180JB81PNC:CAPC1608X90N -> WaterNet26 Library:CAPC1608X90N; symbol WaterNetPowerBoardLibrary:CL10C180JB81PNC -> WaterNet26 Library:CL10C180JB81PNC
- C47, C6, C61, C72: footprint CL21Y105KCYVPNE:CAPC2012X145N -> WaterNet26 Library:CAPC2012X145N; symbol WaterNetPowerBoardLibrary:CL21Y105KCYVPNE -> WaterNet26 Library:CL21Y105KCYVPNE
- C48, C49, C51, C56, C63, C66: footprint CL10A106MA8NRNC:CAPC1608X100N -> WaterNet26 Library:APC1608X100N; symbol WaterNetPowerBoardLibrary:CL10A106MA8NRNC -> WaterNet26 Library:CL10A106MA8NRNC
- C50, C52, C58, C60, C64, C67: footprint CL05B104KA5NNNC:CAPC1005X55N -> WaterNet26 Library:CAPC1005X55N; symbol WaterNetPowerBoardLibrary:CL05B104KA5NNNC -> WaterNet26 Library:CL05B104KA5NNNC
- C55, C57, C59, C62, C65, C73: footprint CL05B102KB5NNNC:CAPC1005X55N -> WaterNet26 Library:CAPC1005X55N; symbol WaterNetPowerBoardLibrary:CL05B102KB5NNNC -> WaterNet26 Library:CL05B102KB5NNNC
- D1, D5: footprint RB070MM-30TR:DIO_RB070MM-30TR -> WaterNet26 Library:DIO_RB070MM-30TR; symbol WaterNetPowerBoardLibrary:RB070MM-30TR -> WaterNet26 Library:RB070MM-30TR
- D11: footprint CLMVC-FKA-CL1D1L71BB7C3C3:LED_CLMVC-FKA-CL1D1L71BB7C3C3 -> WaterNet26 Library:LED_CLMVC-FKA-CL1D1L71BB7C3C3; symbol WaterNetPowerBoardLibrary:CLMVC-FKA-CL1D1L71BB7C3C3 -> WaterNet26 Library:CLMVC-FKA-CL1D1L71BB7C3C3
- F3: footprint 0680L5000-05:FUSC6125X279N -> WaterNet26 Library:FUSC6125X279N; symbol WaterNetPowerBoardLibrary:0680L5000-05 -> WaterNet26 Library:0680L5000-05
- F5: footprint C1F-3:FUSC3215X83N -> WaterNet26 Library:FUSC3215X83N; symbol WaterNetPowerBoardLibrary:C1F-3 -> WaterNet26 Library:C1F-3
- J1, J2: footprint USB4120-03-C_REVA6:GCT_USB4120-03-C_REVA6 -> WaterNet26 Library:GCT_USB4120-03-C_REVA6; symbol WaterNetPowerBoardLibrary:USB4120-03-C_REVA6 -> WaterNet26 Library:USB4120-03-C_REVA6
- J10, J13, J15, J6, J7: footprint XT60-M:AMASS_XT60-M -> WaterNet26 Library:AMASS_XT60-M; symbol WaterNetPowerBoardLibrary:XT60-M -> WaterNet26 Library:XT60-M
- J11, J12, J14: footprint Solderable_100Mil_Jumper -> WaterNet26 Library:Solderable_100Mil_Jumper; symbol WaterNetPowerBoardLibrary:Solderable_100Mil_Jumper -> WaterNet26 Library:Solderable_100Mil_Jumper
- J16, J17, J18, J19, J20, J21: footprint TSW-108-07-F-D:SAMTEC_TSW-108-07-F-D -> WaterNet26 Library:SAMTEC_TSW-108-07-F-D; symbol WaterNetPowerBoardLibrary:TSW-108-07-F-D -> WaterNet26 Library:TSW-108-07-F-D
- J3: symbol WaterNetPowerBoardLibrary:470531000 -> WaterNet26 Library:470531000
- J4: footprint 350761-4:TE_350761-4 -> WaterNet26 Library:TE_350761-4; symbol WaterNetPowerBoardLibrary:350761-4 -> WaterNet26 Library:350761-4
- J5: footprint B2B-PH-K-S:JST_B2B-PH-K-S -> WaterNet26 Library:JST_B2B-PH-K-S; symbol WaterNetPowerBoardLibrary:B2B-PH-K-S -> WaterNet26 Library:B2B-PH-K-S
- J8, J9: footprint SM04B-SRSS-TB:CONN_SM04B-SRSS-TB_JST -> WaterNet26 Library:CONN_SM04B-SRSS-TB_JST; symbol WaterNetPowerBoardLibrary:SM04B-SRSS-TB -> WaterNet26 Library:SM04B-SRSS-TB
- L1, L4, L5: footprint VLS6045EX-150M:IND_VLS6045EX-150M -> WaterNet26 Library:IND_VLS6045EX-150M; symbol WaterNetPowerBoardLibrary:VLS6045EX-150M -> WaterNet26 Library:VLS6045EX-150M
- L2: footprint SRP1265A-220M:IND_SRP1265A-220M -> WaterNet26 Library:ND_SRP1265A-220M; symbol WaterNetPowerBoardLibrary:SRP1265A-220M -> WaterNet26 Library:SRP1265A-220M
- L3: footprint WE-MAPI_5030:WE-MAPI_5030 -> WaterNet26 Library:WE-MAPI_5030; symbol WaterNetPowerBoardLibrary:WE-MAPI_5030 -> WaterNet26 Library:WE-MAPI_5030
- Q1, Q3: footprint SI7149ADP-T1-GE3:POWERPAKSO-8 -> WaterNet26 Library:POWERPAKSO-8; symbol WaterNetPowerBoardLibrary:SI7149ADP-T1-GE3 -> WaterNet26 Library:SI7149ADP-T1-GE3
- R1, R10, R14, R15, R16, R20, R21, R24, R30, R36, R38, R41, R42, R52, R54, R58, R59, R6, R60, R61, R62, R63, R64, R65, R66, R67, R68, R69, R7: footprint ERA6AEB103V:RES_ERA6AEB103V -> WaterNet26 Library:RES_ERA6AEB103V; symbol WaterNetPowerBoardLibrary:ERA6AEB103V -> WaterNet26 Library:ERA6AEB103V
- R11, R2, R5: footprint CSS2725FT1L00:RESC6864X134N -> WaterNet26 Library:RESC6864X134N; symbol WaterNetPowerBoardLibrary:CSS2725FT1L00 -> WaterNet26 Library:CSS2725FT1L00
- R12, R13: footprint CSNL1206FT1L00:RESC3216X90N -> WaterNet26 Library:RESC3216X90N; symbol WaterNetPowerBoardLibrary:CSNL1206FT1L00 -> WaterNet26 Library:CSNL1206FT1L00
- R17, R18, R22, R23: footprint RMCF0603FT5K10:RESC1508X55N -> WaterNet26 Library:RESC1508X55N; symbol WaterNetPowerBoardLibrary:RMCF0603FT5K10 -> WaterNet26 Library:RMCF0603FT5K10
- R19, R26, R37, R43, R8, R9: footprint ERA6AEB304V:RES_ERA6AEB304V -> WaterNet26 Library:RES_ERA6AEB304V; symbol WaterNetPowerBoardLibrary:ERA6AEB304V -> WaterNet26 Library:ERA6AEB304V
- R25: footprint ERJ3EKF1501V:RES_ERJ3EKF1501V -> WaterNet26 Library:RES_ERJ3EKF1501V; symbol WaterNetPowerBoardLibrary:ERJ3EKF1501V -> WaterNet26 Library:ERJ3EKF1501V
- R27: footprint ERA-3AEB4990V:RESC1608X55N -> WaterNet26 Library:RESC1608X55N; symbol WaterNetPowerBoardLibrary:ERA-3AEB4990V -> WaterNet26 Library:ERA-3AEB4990V
- R28, R29: footprint RT0603BRD072K2L:RESC1608X55N -> WaterNet26 Library:RESC1608X55N; symbol WaterNetPowerBoardLibrary:RT0603BRD072K2L -> WaterNet26 Library:RT0603BRD072K2L
- R3, R4: footprint RMCF0805FT2R00:RESC2012X65N -> WaterNet26 Library:RESC2012X65N; symbol WaterNetPowerBoardLibrary:RMCF0805FT2R00 -> WaterNet26 Library:RMCF0805FT2R00
- R31, R32, R33: footprint ERJ3EKF1000V:RES_ERJ3EKF1000V -> WaterNet26 Library:RES_ERJ3EKF1000V; symbol WaterNetPowerBoardLibrary:ERJ3EKF1000V -> WaterNet26 Library:ERJ3EKF1000V
- R34, R35, R55, R56, R57, R91, R92, R93, R94: footprint RMCF0603FT10R0:RESC1508X55N -> WaterNet26 Library:RESC1508X55N; symbol WaterNetPowerBoardLibrary:RMCF0603FT10R0 -> WaterNet26 Library:RMCF0603FT10R0
- R39: footprint ERA6AEB104V:RES_ERA6AEB104V -> WaterNet26 Library:RES_ERA6AEB104V; symbol WaterNetPowerBoardLibrary:ERA6AEB104V -> WaterNet26 Library:ERA6AEB104V
- R40: footprint ERA6AEB3162V:RES_ERA6AEB3162V -> WaterNet26 Library:RES_ERA6AEB3162V; symbol WaterNetPowerBoardLibrary:ERA6AEB3162V -> WaterNet26 Library:ERA6AEB3162V
- R44, R48, R49: footprint ERJ-8BWFR100V:RES_ERJ-8BWFR100V -> WaterNet26 Library:RES_ERJ-8BWFR100V; symbol WaterNetPowerBoardLibrary:ERJ-8BWFR100V -> WaterNet26 Library:ERJ-8BWFR100V
- R45, R46, R47, R50, R51, R53: footprint ERJ2RKF1000X:RES_ERJ2RKF1000X -> WaterNet26 Library:RES_ERJ2RKF1000X; symbol WaterNetPowerBoardLibrary:ERJ2RKF1000X -> WaterNet26 Library:ERJ2RKF1000X
- SW1: footprint CS1213AGF160:CS1213AGF160 -> WaterNet26 Library:CS1213AGF160; symbol WaterNetPowerBoardLibrary:CS1213AGF160 -> WaterNet26 Library:CS1213AGF160
- SW2, SW3: footprint PTS810_SJM_250_SMTR_LFS:SW_PTS810_SJM_250_SMTR_LFS -> WaterNet26 Library:SW_PTS810_SJM_250_SMTR_LFS; symbol WaterNetPowerBoardLibrary:PTS810_SJM_250_SMTR_LFS -> WaterNet26 Library:PTS810_SJM_250_SMTR_LFS
- U1: footprint INA4181A3IPWR:SOP65P640X120-20N -> WaterNet26 Library:SOP65P640X120-20N; symbol WaterNetPowerBoardLibrary:INA4181A3IPWR -> WaterNet26 Library:INA4181A3IPWR
- U10, U11, U9: footprint TPS922051D1DSGR:WSON8_2x2 -> WaterNet26 Library:WSON8_2x2; symbol WaterNetPowerBoardLibrary:TPS922051D1DSGR -> WaterNet26 Library:TPS922051D1DSGR
- U12, U13, U14, U16, U17, U18, U4, U5, U7: footprint BSS123-7-F:SOT95P240X110-3N -> WaterNet26 Library:SOT95P240X110-3N; symbol WaterNetPowerBoardLibrary:BSS123-7-F -> WaterNet26 Library:BSS123-7-F
- U15: footprint Package_SON:WSON-6-1EP_2x2mm_P0.65mm_EP1x1.6mm -> WaterNet26 Library:WSON-6-1EP_2x2mm_P0.65mm_EP1x1.6mm; symbol WaterNetPowerBoardLibrary:TMP117xxDRV -> WaterNet26 Library:TMP117xxDRV
- U2: footprint MIC28514T-E_PHA:CONV_MIC28514T-E_PHA -> WaterNet26 Library:CONV_MIC28514T-E_PHA; symbol WaterNetPowerBoardLibrary:MIC28514T-E_PHA -> WaterNet26 Library:MIC28514T-E_PHA
- U3: footprint MCP2200-I_SO:SOIC20 -> WaterNet26 Library:SOIC20; symbol WaterNetPowerBoardLibrary:MCP2200-I_SO -> WaterNet26 Library:MCP2200-I_SO
- U6: footprint AP62301WU-7:SOT95P280X100-6N -> WaterNet26 Library:SOT95P280X100-6N; symbol WaterNetPowerBoardLibrary:AP62301WU-7 -> WaterNet26 Library:AP62301WU-7
- U8: footprint RF_Module:ESP32-S3-WROOM-1 -> WaterNet26 Library:ESP32-S3-WROOM-1; symbol WaterNetPowerBoardLibrary:ESP32-S3-WROOM-1 -> WaterNet26 Library:ESP32-S3-WROOM-1
- Y1: footprint ECS-120-12-33-AGN-TR:XTAL_ECS-120-12-33-AGN-TR -> WaterNet26 Library:XTAL_ECS-120-12-33-AGN-TR; symbol WaterNetPowerBoardLibrary:ECS-120-12-33-AGN-TR -> WaterNet26 Library:ECS-120-12-33-AGN-TR

Commit message: Changes made to footprints and symbols in existing schematics
Parts:
- C48, C49, C51, C56, C63, C66: footprint WaterNet26 Library:APC1608X100N -> WaterNet26 Library:CAPC1608X100N
Changed lines of the file:
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@@
 			)
 		)
-		(property "Footprint" "WaterNet26 Library:APC1608X100N"
+		(property "Footprint" "WaterNet26 Library:CAPC1608X100N"
 			(at 363.22 525.78 0)
 			(effects
@@
 			)
 		)
-		(property "Footprint" "WaterNet26 Library:APC1608X100N"
+		(property "Footprint" "WaterNet26 Library:CAPC1608X100N"
 			(at 497.84 505.46 0)
 			(effects
@@
 			)
 		)
-		(property "Footprint" "WaterNet26 Library:APC1608X100N"
+		(property "Footprint" "WaterNet26 Library:CAPC1608X100N"
 			(at 363.22 477.52 0)
 			(effects
@@
 			)
 		)
-		(property "Footprint" "WaterNet26 Library:APC1608X100N"
+		(property "Footprint" "WaterNet26 Library:CAPC1608X100N"
 			(at 497.84 408.94 0)
 			(effects
@@
 			)
 		)
-		(property "Footprint" "WaterNet26 Library:APC1608X100N"
+		(property "Footprint" "WaterNet26 Library:CAPC1608X100N"
 			(at 363.22 429.26 0)
 			(effects
@@
 			)
 		)
-		(property "Footprint" "WaterNet26 Library:APC1608X100N"
+		(property "Footprint" "WaterNet26 Library:CAPC1608X100N"
 			(at 497.84 457.2 0)
 			(effects
