File: boat_pcb_v2/WN_power_board/WaterNetPowerBoard.kicad_pcb (KiCad board)
At the start: 2 copper layers, 0.7 x 0.5 mm, 203 parts, among them J1 USB4120-03-C_REVA6, J10 XT60-M, J13 XT60-F, J15 XT60-M, J16 TSW-108-07-F-D, J17 TSW-108-07-F-D, J18 TSW-108-07-F-D, J19 TSW-108-07-F-D, J2 USB4120-03-C_REVA6, J20 TSW-108-07-F-D, J21 TSW-108-07-F-D, J3 4 Pin Fan Header, J4 350761-4, J5 B2B-PH-K-S, J6 XT60-F, J7 XT60-M, J8 QWIIC, J9 QWIIC, Q1 SI7149ADP-T1-GE3, Q3 SI7149ADP-T1-GE3, SW2 Push Button, SW3 Push Button, U1 INA4181A3IPWR, U10 TPS922051D1DSGR, U11 TPS922051D1DSGR, U12 BSS123-7-F, U13 BSS123-7-F, U14 BSS123-7-F, U15 TMP117xxDRV, U16 BSS123-7-F, U17 BSS123-7-F, U18 BSS123-7-F, U2 MIC28514T-E_PHA, U3 MCP2200-I_SO, U4 BSS123-7-F, U5 BSS123-7-F, U6 AP62301WU-7, U7 BSS123-7-F, U8 ESP32-S3-WROOM-1, U9 TPS922051D1DSGR, Y1 ECS-120-12-33-AGN-TR

Commit message: minor updates related to board layout
Parts:
- R11, R2, R5, U3: moved to B.Cu
- moved U3 0.66 mm to (124.9, 45.0), turned to 180 degrees
- turned R11 to 180 degrees
- turned R2 to 180 degrees
- turned R5 to 180 degrees
