File: boat_pcb_v2/WN_sensor_board/sensor_board.kicad_pcb (KiCad board)
At the start: 2 copper layers, 0.7 x 0.5 mm, 103 parts, among them J1 MSD-4-A, J10 PPTC031LFBN-RC, J11 RFPC-SMA28-F, J12 PPTC031LFBN-RC, J13 PPTC031LFBN-RC, J14 RFPC-SMA28-F, J15 USB4120-03-C_REVA6, J16 USB4120-03-C_REVA6, J2 RFPC-SMA28-F, J3 RFPC-SMA28-F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

Commit message: Began Jetson board
Parts:
- added C40: 0.1uF 25V, WaterNet26 Footprints:CAPC2012X95N, F.Cu at (184.6, 99.7)
- added C41: 0.1uF 25V, WaterNet26 Footprints:CAPC2012X95N, F.Cu at (184.6, 102.7)
- added C42: 0.1uF 25V, WaterNet26 Footprints:CAPC2012X95N, F.Cu at (184.6, 105.6)
- added J17: PPTC031LFBN-RC, WaterNet26 Footprints:CONN_PPTC031_SUL, F.Cu at (169.7, 101.3)
- added J18: PPTC031LFBN-RC, WaterNet26 Footprints:CONN_PPTC031_SUL, F.Cu at (169.7, 106.5)
- added J20: TSW-108-07-F-D, WaterNet26 Footprints:SAMTEC_TSW-108-07-F-D, F.Cu at (173.8, 81.7)
- added J21: TSW-108-07-F-D, WaterNet26 Footprints:SAMTEC_TSW-108-07-F-D, F.Cu at (173.8, 88.3)
- added J22: TSW-108-07-F-D, WaterNet26 Footprints:SAMTEC_TSW-108-07-F-D, F.Cu at (173.8, 95.0)
- added J4: RFPC-SMA28-F, WaterNet26 Footprints:GRADCONN_RFPC-SMA28-F, F.Cu at (177.8, 102.9)
- added R1: ERA6AEB104V, WaterNet26 Footprints:RES_ERA6AEB104V, F.Cu at (187.3, 79.8)
- added R2: ERA6AEB104V, WaterNet26 Footprints:RES_ERA6AEB104V, F.Cu at (187.3, 82.6)
- added R37: ERA6AEB304V, WaterNet26 Footprints:RES_ERA6AEB304V, F.Cu at (187.3, 85.4)
- added R38: 10K, WaterNet26 Footprints:RES_ERA6AEB103V, F.Cu at (187.3, 88.2)
- added R42: 10K, WaterNet26 Footprints:RES_ERA6AEB103V, F.Cu at (187.3, 91.0)
- added R43: ERA6AEB304V, WaterNet26 Footprints:RES_ERA6AEB304V, F.Cu at (187.3, 93.8)
- added U8: BSS123-7-F, WaterNet26 Footprints:SOT95P240X110-3N, F.Cu at (189.0, 100.4)
- added U9: BSS123-7-F, WaterNet26 Footprints:SOT95P240X110-3N, F.Cu at (189.0, 104.5)
- PS1, PS2, PS3, PS4: footprint WaterNet26 Footprints:CONV_MIC28514T-E_PHA -> WaterNet26 Footprints:CONV_TBA_1-0310
- moved L6 0.31 mm to (149.7, 94.6)
- moved R33 0.18 mm to (154.0, 94.5)
Connections:
- U2 pad 23: unconnected-(U2-IO21-Pad23) -> /OFFBOARD_DET
- U2 pad 3: unconnected-(U2-EN-Pad3) -> /SYS_RST
- U2 pad 38: unconnected-(U2-IO2-Pad38) -> /IO2
- U2 pad 39: unconnected-(U2-IO1-Pad39) -> /IO1
- U2 pad 4: unconnected-(U2-IO4-Pad4) -> /LEAK_DET_S
- U2 pad 5: unconnected-(U2-IO5-Pad5) -> /LEAK_DET_OFFBD_S
Other:
- copper layers 2 -> 4
