File: boat_pcb_v2/WN_sensor_board/sensor_board.kicad_sch (KiCad schematic)
At the start: 47 parts, among them J1 PCB.SMAFRA.HT, J2 USB_C_Receptacle_USB2.0_16P, J3 USB_C_Receptacle_USB2.0_16P, U1 MAX14933ASE_T, U2 ESP32-S3-WROOM-1-N8, U3 MCP2221-I_ST, U4 AP62301WU-7

Commit message: Updated submodule
Parts:
- added C16, C18, C19, C20, C21, C24, C25: 10µ, 25V, Capacitor_SMD:C_0603_1608Metric_Pad1.08x0.95mm_HandSolder, symbol WN_sensor_board:C
- added J10, J12, J13, J5, J6, J7, J8, J9: PPTC031LFBN-RC, CONN_PPTC031_SUL, symbol WN_sensor_board:PPTC031LFBN-RC
- added J11, J14, J4: PCB.SMAFRA.HT, CONN_PCB.SMAFRA_TAL, symbol WN_sensor_board:PCB.SMAFRA.HT
- added PS2, PS3, PS4: TBA_1-0310, TBA_1-0310:CONV_TBA_1-0310, symbol WN_sensor_board:TBA_1-0310
- added Q1: IPD90N04S4-05, IPD90N04S405, symbol WN_sensor_board:IPD90N04S4-05
- added R12: R, symbol WN_sensor_board:R
- added R13, R14, R15, R16, R17, R18, R19, R21: 10k, symbol WN_sensor_board:R
- added U5, U6, U7: MAX14933ASE_T, MAX14933ASE_T:SOIC127P600X175-16N, symbol WN_sensor_board:MAX14933ASE_T
- C1, C10, C11, C12, C13, C14, C15, C17, C2, C22, C23, C3, C4, C5, C6, C7, C8: symbol Device:C -> WN_sensor_board:C
- C9: symbol WaterNet26:GCM188R71E224KA55D -> WN_sensor_board:GCM188R71E224KA55D
- D1: symbol Power_Protection:USBLC6-2SC6 -> WN_sensor_board:USBLC6-2SC6
- D1, D2, D3: symbol Device:D_Schottky -> WN_sensor_board:D_Schottky
- J1: symbol WaterNet26:PCB.SMAFRA.HT -> WN_sensor_board:PCB.SMAFRA.HT
- J2, J3: symbol Connector:USB_C_Receptacle_USB2.0_16P -> WN_sensor_board:USB_C_Receptacle_USB2.0_16P
- L1, L3, L4: symbol Device:L -> WN_sensor_board:L
- PS1: symbol WaterNet26:TBA_1-0310 -> WN_sensor_board:TBA_1-0310
- R1, R10, R11, R2, R20, R3, R4, R5, R6, R7, R8, R9: symbol Device:R -> WN_sensor_board:R
- S1, S2: symbol push_button:TS04-66-50-BK-160-SMT-TR -> WN_sensor_board:TS04-66-50-BK-160-SMT-TR
- U1: symbol WaterNet26:MAX14933ASE_T -> WN_sensor_board:MAX14933ASE_T
- U2: symbol WaterNet26:ESP32-S3-WROOM-1-N8 -> WN_sensor_board:ESP32-S3-WROOM-1-N8
- U3: symbol WaterNet26:MCP2221-I_ST -> WN_sensor_board:MCP2221-I_ST_1
- U4: symbol Regulators:AP62301WU-7 -> WN_sensor_board:AP62301WU-7
Connections:
- net GNDB is gone; now on net GND: U1.16 (GNDB), U1.9 (GNDB)
- net +3V3: now also Q1.3 (S), R12.2
- net GND: now also PS1.3 (-VOUT), C16.1, C18.2, C19.1, C20.2, C21.1, C24.2, C25.1, J10.1, J13.1, J5.1, J8.1, PS2.1 (-VIN(GND)), PS2.3 (-VOUT), PS3.1 (-VIN(GND)), PS3.3 (-VOUT), PS4.1 (-VIN(GND)), PS4.3 (-VOUT), U5.1 (GNDA), U5.10 (I.C.), U5.15 (I.C.), U5.16 (GNDB), U5.2 (I.C.), U5.7 (GNDA), U5.8 (I.C.), U5.9 (GNDB), U6.1 (GNDA), U6.10 (I.C.), U6.15 (I.C.), U6.16 (GNDB), U6.2 (I.C.), U6.7 (GNDA), U6.8 (I.C.), U6.9 (GNDB), U7.1 (GNDA), U7.10 (I.C.), U7.15 (I.C.), U7.16 (GNDB), U7.2 (I.C.), U7.7 (GNDA), U7.8 (I.C.), U7.9 (GNDB)
- net SCL: now also U5.5 (I/OA1), U6.5 (I/OA1), U7.5 (I/OA1)
- net SDA: now also U5.6 (I/OA2), U6.6 (I/OA2), U7.6 (I/OA2)
- net USB_D+: now also U2.14 (IO20); no longer U2.20 (IO12)
- net USB_D-: now also U2.13 (IO19); no longer U2.19 (IO11)
- net SEN_POW: now reaches U2.26 (IO45)
- net SEN_POW: now also Q1.1 (G), R12.1
- net PRB1: now reaches J1.1
- net PRB1: now also J6.2
- net PGND1: now reaches J1.2
- net PGND1: now also J1.3, J1.4, J1.5, J6.3
- net +3V3_S: now reaches C15.1, PS1.2 (+VIN(VCC))
- net +3V3_S: now also U1.3 (VDDA), C18.1, C20.1, C24.1, PS2.2 (+VIN(VCC)), PS3.2 (+VIN(VCC)), PS4.2 (+VIN(VCC)), Q1.2 (D), U5.3 (VDDA), U6.3 (VDDA), U7.3 (VDDA)
- net ISO_SDA_1: now reaches U1.11 (I/OB2)
- net ISO_SDA_1: now also J5.2, R14.2
- net ISO_SCL_1: now reaches U1.12 (I/OB1)
- net ISO_SCL_1: now also J5.3, R13.2
- net ISO_3V3: now reaches U1.14 (VDDB)
- net ISO_3V3: now also PS1.4 (+VOUT), C16.2, C19.2, C21.2, C25.2, J12.1, J6.1, J7.1, J9.1, PS2.4 (+VOUT), PS3.4 (+VOUT), PS4.4 (+VOUT), R13.1, R14.1, R15.1, R16.1, R17.1, R18.1, R19.1, R21.1, U5.14 (VDDB), U6.14 (VDDB), U7.14 (VDDB)
- new net ISO_SCL_2: J8.3, R15.2, U5.12 (I/OB1)
- new net ISO_SCL_3: J10.3, R17.2, U6.12 (I/OB1)
- new net ISO_SCL_4: J13.3, R19.2, U7.12 (I/OB1)
- new net ISO_SDA_2: J8.2, R16.2, U5.11 (I/OB2)
- new net ISO_SDA_3: J10.2, R18.2, U6.11 (I/OB2)
- new net ISO_SDA_4: J13.2, R21.2, U7.11 (I/OB2)
- new net PGND2: J4.2, J4.3, J4.4, J4.5, J7.3
- new net PGND3: J11.2, J11.3, J11.4, J11.5, J9.3
- new net PGND4: J12.3, J14.2, J14.3, J14.4, J14.5
- new net PRB2: J4.1, J7.2
- new net PRB3: J11.1, J9.2
- new net PRB4: J12.2, J14.1
- no-connect marks 8 -> 11
Other:
- note added: "Atlas Sensor 1"
- note added: "Atlas Sensor 2"
- note added: "Atlas Sensor 3"
- note added: "Atlas Sensor 4"
- note added: "Power Switch for Sensors"
- moved on the sheet: C1, C15, C2, C3, C4, C6, D1, J1, J2, L3, PS1, R1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

Commit message: Changes made to footprints and symbols in existing schematics
Parts:
- removed C3, C4, C7, C8: 1µ, 25V, Capacitor_SMD:C_0603_1608Metric_Pad1.08x0.95mm_HandSolder, symbol WN_sensor_board:C
- removed C9: .22µF, GCM188R71E224KA55D:CAPC1608X90N, symbol WN_sensor_board:GCM188R71E224KA55D
- removed D1: USBLC6-2SC6, Package_TO_SOT_SMD:SOT-23-6, symbol WN_sensor_board:USBLC6-2SC6
- removed J1, J11, J14, J4: PCB.SMAFRA.HT, CONN_PCB.SMAFRA_TAL, symbol WN_sensor_board:PCB.SMAFRA.HT
- removed J2, J3: USB_C_Receptacle_USB2.0_16P, Connector_USB:USB_C_Plug_ShenzhenJingTuoJin_918-118A2021Y40002_Vertical, symbol WN_sensor_board:USB_C_Receptacle_USB2.0_16P
- removed L3, L4: 3.3µ, WaterNet26_Parts_Lib:INDC1608X95N, symbol WN_sensor_board:L
- removed Q1: IPD90N04S4-05, IPD90N04S405, symbol WN_sensor_board:IPD90N04S4-05
- removed R2, R3, R6, R7, R8: 5.1k, Resistor_SMD:R_0603_1608Metric, symbol WN_sensor_board:R
- removed U3: MCP2221-I_ST, MCP2221-I_ST:SOP65P640X120-14N, symbol WN_sensor_board:MCP2221-I_ST_1
- added C26, C27, C28, C9: 1µ, 25V, WaterNet26 Footprints:CAPC2012X145N, symbol Device:C
- added C29: 10µ, 25V, WaterNet26 Footprints:CAPC2012X145N, symbol Device:C
- added C33, C34, C68, C69, C76: 0.1uF 25V, WaterNet26 Footprints:CAPC2012X95N, symbol WaterNet26 Library:CL21B104KACNNNC
- added C35: 10uF 25V, WaterNet26 Footprints:CAPC2012X145N, symbol WaterNet26 Library:CL21A106KAYNNNE
- added C36, C37: 18pF, WaterNet26 Footprints:CAPC1608X90N, symbol WaterNet26 Library:CL10C180JB81PNC
- added D11: CLMVC-FKA-CL1D1L71BB7C3C3, WaterNet26 Footprints:LED_CLMVC-FKA-CL1D1L71BB7C3C3, symbol WaterNet26 Library:CLMVC-FKA-CL1D1L71BB7C3C3
- added D4: USBLC6-2SC6, Package_TO_SOT_SMD:SOT-23-6, symbol Power_Protection:USBLC6-2SC6
- added J1: MSD-4-A, WaterNet26 Footprints:CUI_MSD-4-A, symbol WaterNet26 Library:MSD-4-A
- added J11, J14, J2, J3: RFPC-SMA28-F, WaterNet26 Footprints:GRADCONN_RFPC-SMA28-F, symbol WaterNet26 Library:RFPC-SMA28-F
- added J15, J16: USB4120-03-C_REVA6, WaterNet26 Footprints:GCT_USB4120-03-C_REVA6, symbol WaterNet26 Library:USB4120-03-C_REVA6
- added L5, L6: 3.3µ, WaterNet26 Footprints:INDC1608X95N, symbol Device:L
- added MOSFET1: IRFR5505TRPBF, WaterNet26 Footprints:PG-TO252AA_INF, symbol WaterNet26 Library:IRFR5505TRPBF
- added R22, R23, R25, R26: 5.1K, WaterNet26 Footprints:RESC1508X55N, symbol WaterNet26 Library:RMCF0603FT5K10
- added R24, R66, R67, R68: 10K, WaterNet26 Footprints:RES_ERA6AEB103V, symbol WaterNet26 Library:ERA6AEB103V
- added R27: 10k, WaterNet26 Footprints:RES_ERA6AEB103V, symbol Device:R
- added R31, R32, R33: 100 Ohm, WaterNet26 Footprints:RES_ERJ3EKF1000V, symbol WaterNet26 Library:ERJ3EKF1000V
- added U16, U17, U18, U19: BSS123-7-F, WaterNet26 Footprints:SOT95P240X110-3N, symbol WaterNet26 Library:BSS123-7-F
- added U3: MCP2200-I_SO, WaterNet26 Footprints:SOIC20, symbol WaterNet26 Library:MCP2200-I_SO
- added Y1: ECS-120-12-33-AGN-TR, WaterNet26 Footprints:XTAL_ECS-120-12-33-AGN-TR, symbol WaterNet26 Library:ECS-120-12-33-AGN-TR
- C1: value 0.1µ -> 0.1µ, 25V; footprint (none) -> WaterNet26 Footprints:CAPC2012X95N; symbol WN_sensor_board:C -> Device:C
- C10, C14, C17, C22, C5: footprint Capacitor_SMD:C_0603_1608Metric_Pad1.08x0.95mm_HandSolder -> WaterNet26 Footprints:CAPC2012X95N; symbol WN_sensor_board:C -> Device:C
- C11, C13, C15, C16, C18, C19, C20, C21, C23, C24, C25: footprint Capacitor_SMD:C_0603_1608Metric_Pad1.08x0.95mm_HandSolder -> WaterNet26 Footprints:CAPC2012X145N; symbol WN_sensor_board:C -> Device:C
- C12: value 47µ, 6.3V -> 47µ, 25V; footprint Capacitor_SMD:C_0603_1608Metric_Pad1.08x0.95mm_HandSolder -> WaterNet26 Footprints:CAPC3216X180N; symbol WN_sensor_board:C -> Device:C
- C2: footprint (none) -> WaterNet26 Footprints:CAPC1608X105N; symbol WN_sensor_board:C -> WaterNet26 Library:CL10A226MP8NUNE; A_max (none) -> 1.05; A_min (none) -> 1.05; A_nom (none) -> 1.05; Availability (none) -> In Stock; Check_prices (none) -> https://www.snapeda.com/parts/CL10A226MP8NUNE/Samsung/view-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; D_max (none) -> 1.85; D_min (none) -> 1.35; D_nom (none) -> 1.6; Description_1 (none) -> Cap Ceramic 22uF 10V X5R 20% Pad SMD 0603 85°C Low ESR T/R; E_max (none) -> 1.05; E_min (none) -> 0.55; E_nom (none) -> 0.8; L1_max (none) -> 0.5; L1_min (none) -> 0.1; L1_nom (none) -> 0.3; L_max (none) -> 0.5; L_min (none) -> 0.1; L_nom (none) -> 0.3; MANUFACTURER (none) -> Samsung Electro-Mechanics; MF (none) -> Samsung Electro-Mechanics; MP (none) -> CL10A226MP8NUNE; Package (none) -> SMD-2 Samsung; Price (none) -> None; STANDARD (none) -> IPC 7351B; SnapEDA_Link (none) -> https://www.snapeda.com/parts/CL10A226MP8NUNE/Samsung/view-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
- C6: value C -> 1µF; footprint (none) -> WaterNet26 Footprints:CAPC2012X145N; symbol WN_sensor_board:C -> Device:C
- D1, D2, D3: value D_Schottky -> RB070MM-30TR; footprint WaterNet26_Parts_Lib:SMB -> WaterNet26 Footprints:SMB; symbol WN_sensor_board:D_Schottky -> WaterNet26 Library:RB070MM-30TR
- J10, J12, J13, J5, J6, J7, J8, J9: footprint CONN_PPTC031_SUL -> WaterNet26 Footprints:CONN_PPTC031_SUL; symbol WN_sensor_board:PPTC031LFBN-RC -> WaterNet26 Library:PPTC031LFBN-RC
- L1: footprint WaterNet26_Parts_Lib:INDC1608X95N -> WaterNet26 Footprints:INDC1608X95N; symbol WN_sensor_board:L -> Device:L
- PS1, PS2, PS3, PS4: footprint TBA_1-0310:CONV_TBA_1-0310 -> WaterNet26 Footprints:CONV_MIC28514T-E_PHA; symbol WN_sensor_board:TBA_1-0310 -> WaterNet26 Library:TBA_1-0310
- R1, R12, R5: value R -> 10k; footprint (none) -> WaterNet26 Footprints:RES_ERA6AEB103V; symbol WN_sensor_board:R -> Device:R
- R10: footprint Resistor_SMD:R_0603_1608Metric -> WaterNet26 Footprints:RES_ERA6AEB3162V; symbol WN_sensor_board:R -> Device:R
- R11: footprint Resistor_SMD:R_0603_1608Metric -> WaterNet26 Footprints:RES_ERA6AEB103V; symbol WN_sensor_board:R -> Device:R
- R13, R14, R15, R16, R17, R18, R19, R21: footprint (none) -> WaterNet26 Footprints:RES_ERA6AEB103V; symbol WN_sensor_board:R -> Device:R
- R20, R4, R9: footprint Resistor_SMD:R_0603_1608Metric -> WaterNet26 Footprints:RES_ERA6AEB104V; symbol WN_sensor_board:R -> Device:R
- S1, S2: footprint TS04-66-50-BK-160-SMT-TR:SW_TS04-66-50-BK-160-SMT-TR -> WaterNet26 Footprints:SW_TS04-66-50-BK-160-SMT-TR; symbol WN_sensor_board:TS04-66-50-BK-160-SMT-TR -> WaterNet26 Library:TS04-66-50-BK-160-SMT-TR
- U1, U5, U6, U7: footprint MAX14933ASE_T:SOIC127P600X175-16N -> WaterNet26 Footprints:SOIC127P600X175-16N; symbol WN_sensor_board:MAX14933ASE_T -> WaterNet26 Library:MAX14933ASE_T
- U2: footprint ESP32-S3-WROOM-1-N8:XCVR_ESP32-S3-WROOM-1-N8 -> WaterNet26 Footprints:XCVR_ESP32-S3-WROOM-1-N8; symbol WN_sensor_board:ESP32-S3-WROOM-1-N8 -> WaterNet26 Library:ESP32-S3-WROOM-1-N8
- U4: footprint WaterNet26_Parts_Lib:SOT95P280X100-6N -> WaterNet26 Footprints:SOT95P280X100-6N; symbol WN_sensor_board:AP62301WU-7 -> WaterNet26 Library:AP62301WU-7
Connections:
- net GPIO0 is gone; now on net MODE: R1.2, U2.27 (IO0)
- net +12V: no longer D1.2 (A)
- net +3V3: now also C2.2, C33.1, C35.1, D11.1, MOSFET1.2, R24.2, R27.1, U3.1 (VDD); no longer C2.1, R12.2
- net +3V3_S: now also MOSFET1.3
- net +VBUSF_1: now also C28.1, L6.2; no longer D2.2 (A)
- net +VBUSF_2: now also C26.1, L5.2, U3.17 (VUSB); no longer D3.2 (A)
- net MODE: no longer C5.1, R4.2, S1.1, S1.3
- net PGND1: now also J14.G1, J14.G2, J14.G3, J14.G4
- net PGND2: now also J11.G1, J11.G2, J11.G3, J11.G4
- net PGND3: now also J2.G1, J2.G2, J2.G3, J2.G4
- net PGND4: now also J3.G1, J3.G2, J3.G3, J3.G4
- net PRB1: now also J14.1
- net PRB2: now also J11.1
- net PRB3: now also J2.1
- net PRB4: now also J3.1
- net SEN_POW: now also U19.1 (G)
- net USB_D+: now also D4.4 (I/O2)
- net USB_D-: now also D4.6 (I/O1)
- net VSEL: no longer D1.1 (K), D2.1 (K), D3.1 (K)
- net MOSI: now reaches U2.12 (IO8)
- net MOSI: now also J1.3 (CMD)
- net RGB_R: now reaches U2.16 (IO46)
- net RGB_R: now also C76.1, R68.2, U18.1 (G)
- net MISO: now reaches U2.17 (IO9)
- net MISO: now also J1.7 (DAT0)
- net SCK: now reaches U2.18 (IO10)
- net SCK: now also J1.5 (CLK)
- net CS: now reaches U2.19 (IO11)
- net CS: now also J1.2 (CD/DAT3)
- net SD_DET: now reaches U2.20 (IO12)
- net SD_DET: now also J1.CD
- net SYS_RST: now reaches C6.1, R5.2
- net SYS_RST: now also C5.1, R4.2, S1.1, S1.3; no longer U2.3 (EN)
- net RGB_G: now reaches U2.31 (IO38)
- net RGB_G: now also C69.1, R66.2, U17.1 (G)
- net USB_CTS: now reaches U2.8 (IO15)
- net USB_CTS: now also U3.13 (~{CTS})
- net USB_RTS: now reaches U2.9 (IO16)
- net USB_RTS: now also U3.11 (~{RTS})
- net GND renamed COVER_GND
- net COVER_GND: now also C2.1, R12.2, C26.2, C27.2, C28.2, C29.1, C33.2, C34.2, C35.2, C36.1, C37.1, C68.2, C69.2, C76.2, C9.2, D4.2 (GND), J1.6 (VSS), J1.G1 (COVER_GND), J1.G2 (COVER_GND), J1.G3 (COVER_GND), J1.G4 (COVER_GND), J15.A1 (GND_A), J15.A12 (GND_A), J15.B1 (GND_B), J15.B12 (GND_B), J15.S1 (SHIELD), J15.S2 (SHIELD), J15.S3 (SHIELD), J15.S4 (SHIELD), J16.A1 (GND_A), J16.A12 (GND_A), J16.B1 (GND_B), J16.B12 (GND_B), J16.S1 (SHIELD), J16.S2 (SHIELD), J16.S3 (SHIELD), J16.S4 (SHIELD), R22.1, R23.1, R25.1, R26.1, R66.1, R67.1, R68.1, U16.2 (S), U17.2 (S), U18.2 (S), U19.2 (S), U3.20 (VSS), Y1.2 (GND), Y1.4 (GND); no longer C2.2
- net MTCK renamed RGB_B
- net RGB_B: now also C68.1, R67.2, U16.1 (G)
- net MTDI: no longer names the net of U2.34 (IO41)
- net MTDO: no longer names the net of U2.33 (IO40)
- net MTMS: no longer names the net of U2.35 (IO42)
- net PWM0: no longer names the net of U2.4 (IO4)
- net PWM1: no longer names the net of U2.5 (IO5)
- net PWM2: no longer names the net of U2.6 (IO6)
- net PWM3: no longer names the net of U2.7 (IO7)
- net UORXD renamed USB_RX
- net USB_RX: now also U3.12 (RX)
- net UOTXD renamed USB_TX
- net USB_TX: now also U3.10 (TX)
- new net: R31.1, U16.3 (D)
- new net: J15.B5 (CC2), R23.2
- new net: C29.2, C34.1, J1.4 (VDD)
- new net: C37.2, U3.3 (OSC2), Y1.3 (OUT/IN)
- new net: MOSFET1.1, R27.2, U19.3 (D)
- new net: C36.2, U3.2 (OSC1), Y1.1 (IN/OUT)
- new net: R24.1, U3.4 (RST)
- new net: R33.1, U18.3 (D)
- new net: J16.A5 (CC1), R25.2
- new net: D4.3 (I/O2), J16.A6 (D1+), J16.B6 (D2+)
- new net: D4.1 (I/O1), J16.A7 (D1-), J16.B7 (D2-)
- new net: J16.B5 (CC2), R26.2
- new net: D11.4, R33.2
- new net: D11.2, R31.2
- new net: J15.A5 (CC1), R22.2
- new net: R32.1, U17.3 (D)
- new net: D11.3, R32.2
- new net USB_D2+: J15.A6 (D1+), J15.B6 (D2+), U3.19 (D+)
- new net USB_D2-: J15.A7 (D1-), J15.B7 (D2-), U3.18 (D-)
- new net VBUS_A: C27.1, C9.1, J15.A4 (VBUS_A), J15.A9 (VBUS_A), J15.B4 (VBUS_B), J15.B9 (VBUS_B), J16.A4 (VBUS_A), J16.A9 (VBUS_A), J16.B4 (VBUS_B), J16.B9 (VBUS_B), L5.1, L6.1
- no-connect marks 11 -> 17
Other:
- note added: "MicroSD Card Reader"
- note added: "Onboard RGB LED"
- moved on the sheet: C1, C6, R1, R12, R5

Commit message: Finished Sensor Board
Parts:
- removed C6: 1µF, WaterNet26 Footprints:CAPC2012X145N, symbol Device:C
- removed R1, R5: 10k, WaterNet26 Footprints:RES_ERA6AEB103V, symbol Device:R
- added C40, C41: 0.1uF 25V, WaterNet26 Footprints:CAPC2012X95N, symbol WaterNet26 Library:CL21B104KACNNNC
- added J17, J18: PPTC031LFBN-RC, WaterNet26 Footprints:CONN_PPTC031_SUL, symbol WaterNet26 Library:PPTC031LFBN-RC
- added J20, J21: TSW-108-07-F-D, WaterNet26 Footprints:SAMTEC_TSW-108-07-F-D, symbol WaterNet26 Library:TSW-108-07-F-D
- added J4: RFPC-SMA28-F, WaterNet26 Footprints:GRADCONN_RFPC-SMA28-F, symbol WaterNet26 Library:RFPC-SMA28-F
- added R1, R2: ERA6AEB104V, WaterNet26 Library:RES_ERA6AEB104V, symbol WaterNet26 Library:ERA6AEB104V
- added R37, R43: ERA6AEB304V, WaterNet26 Footprints:RES_ERA6AEB304V, symbol WaterNet26 Library:ERA6AEB304V
- added R38, R42: 10K, WaterNet26 Footprints:RES_ERA6AEB103V, symbol WaterNet26 Library:ERA6AEB103V
- added U8, U9: BSS123-7-F, WaterNet26 Footprints:SOT95P240X110-3N, symbol WaterNet26 Library:BSS123-7-F
Connections:
- net +3V3: now also J20.14, J20.16, J21.14, J21.16, R38.1, R42.1
- net +3V3_S: now also J17.1
- net COVER_GND: now also C40.1, C41.1, J18.1, J20.15, J21.15, R2.1, R37.1, R43.1, U8.2 (S), U9.2 (S)
- net CS: now also J20.04
- net MISO: now also J20.02
- net MODE: now also J20.03
- net MOSI: now also J20.13
- net RGB_B: now also J21.07
- net RGB_G: now also J21.05
- net RGB_R: now also J21.09
- net SCK: now also J20.06
- net SCL: now also J18.3, J20.10
- net SDA: now also J18.2, J20.08
- net SD_DET: now also J21.02
- net SEN_POW: now also J21.11
- net SYS_RST: now also U2.3 (EN), J20.01
- net USB_CTS: now also J20.12
- net USB_D+: now also J21.03
- net USB_D-: now also J21.01
- net USB_RTS: now also J21.13
- net USB_RX: now also J20.05
- net USB_TX: now also J20.07
- net OFFBOARD_DET: now reaches U2.23 (IO21)
- net OFFBOARD_DET: now also J21.04, R1.1, R2.2
- net LEAK_DET_S: now reaches U2.4 (IO4)
- net LEAK_DET_S: now also J20.09, R42.2, U8.3 (D)
- net LEAK_DET_OFFBD_S: now reaches U2.5 (IO5)
- net LEAK_DET_OFFBD_S: now also J20.11, R38.2, U9.3 (D)
- new net EXT_SIG: J21.06, R1.2
- new net LEAK_DET: C41.2, R43.2, U8.1 (G)
- new net LEAK_DET_OFFBD: C40.2, R37.2, U9.1 (G)
- new net TEMP_PRB: J17.2, J4.1
- new net TEMP_PRB_GND: J17.3, J4.G1, J4.G2, J4.G3, J4.G4
Other:
- note added: "Altas Temp Sens"
- note added: "External Power Det"
- note added: "Leak Detection"
- moved on the sheet: C1, C68, C69, C76, D11, MOSFET1, R12, R27, R31, R32, R33, R66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

Commit message: Began Jetson board
Parts:
- added C42: 0.1uF 25V, WaterNet26 Footprints:CAPC2012X95N, symbol WaterNet26 Library:CL21B104KACNNNC
- added J22: TSW-108-07-F-D, WaterNet26 Footprints:SAMTEC_TSW-108-07-F-D, symbol WaterNet26 Library:TSW-108-07-F-D
- PS1, PS2, PS3, PS4: footprint WaterNet26 Footprints:CONV_MIC28514T-E_PHA -> WaterNet26 Footprints:CONV_TBA_1-0310
- R1, R2: footprint WaterNet26 Library:RES_ERA6AEB104V -> WaterNet26 Footprints:RES_ERA6AEB104V
Connections:
- net +12V: now also D1.1
- net +VBUSF_1: now also D2.1
- net +VBUSF_2: now also D3.1
- net COVER_GND: now also C42.1
- net SEN_POW: now also C42.2
- net VSEL: now also D1.2, D2.2, D3.2
- net IO2: now reaches U2.38 (IO2)
- net IO1: now reaches U2.39 (IO1)
