File: boat_pcb_v2/WN_jetson_board/jetson_board.kicad_sch (KiCad schematic)
At the start: 15 parts, among them J2 Conn_02x20_Counter_Clockwise, U1 MIC28514T-E_PHA

Commit message: Adafruit breakout, USBC, Regulator
Parts:
- removed J2: Conn_02x20_Counter_Clockwise, symbol Connector_Generic:Conn_02x20_Counter_Clockwise
- added C10: 47µF, WaterNet Footprints:CAPC3216X180N, symbol WaterNet Library:C3216X5R1E476M160AC
- added C11: 10µF, WaterNet Footprints:CAPC2012X145N, symbol WaterNet Library:CL21A106KAYNNNE
- added C12: 0.1µF, WaterNet Footprints:CAPC2012X95N, symbol WaterNet Library:CL21B104KACNNNC
- added C14, C15: 0.1uF 100V, WaterNet Footprints:CAPC2012X135N, symbol WaterNet26 Library:CL21B104KCFSFNE
- added C16, C17, C18, C19: 1µF 100V, WaterNet Footprints:CAPC2012X145N, symbol WaterNet Library:CL21Y105KCYVPNE
- added C9: 10nF, WaterNet Footprints:CAPC1608X90N, symbol WaterNet Library:CL10B103KB8NNNC
- added J1, J3: 6130XX11821_61300811821, WaterNet Footprints:61300811821, symbol WaterNet Library:6130XX11821_61300811821
- added J4: PPTC041LFBN-RC, WaterNet Footprints:SULLINS_PPTC041LFBN-RC, symbol WaterNet Library:PPTC041LFBN-RC
- added J5, J7: USB4120-03-C_REVA6, WaterNet Footprints:GCT_USB4120-03-C_REVA6, symbol WaterNet Library:USB4120-03-C_REVA6
- added J6: Conn_02x20_Odd_Even, symbol Connector_Generic:Conn_02x20_Odd_Even
- added L1, L2, L3: 6.8µH, 8A, WaterNet Footprints:IND_PA4342.682NLT, symbol WaterNet Library:PA4342.682NLT
- added R24, R25, R26, R27: 5.1K, WaterNet26 Footprints:RESC1508X55N, symbol WaterNet26 Library:RMCF0603FT5K10
- added R6, R7: 10k, WaterNet Footprints:RES_ERA6AEB103V, symbol WaterNet Library:ERA6AEB103V
- added R8: 1.37k 0.5%, WaterNet Footprints:RESC1608X55N, symbol WaterNet Library:RT0603DRD071K37L
- added R9: 1.42k, WaterNet Footprints:RESC1608X55N, symbol WaterNet Library:RT0603BRD071K42L
- C1: footprint WaterNet26 Library:CAPC3225X280N -> WaterNet Footprints:CAPC3225X280N
- C2: footprint WaterNet26 Library:CAPC2012X135N -> WaterNet Footprints:CAPC2012X135N
- C3, C6, C8: footprint WaterNet26 Library:CAPC2012X145N -> WaterNet Footprints:CAPC2012X145N
- C4: footprint WaterNet26 Library:CAPC1608X90N -> WaterNet Footprints:CAPC1608X90N
- C5, C7: footprint WaterNet26 Library:CAPC2012X95N -> WaterNet Footprints:CAPC2012X95N
- R1, R2, R3: footprint WaterNet26 Library:RES_ERA6AEB304V -> WaterNet Footprints:RES_ERA6AEB304V
- R4, R5: footprint WaterNet26 Library:RESC2012X65N -> WaterNet Footprints:RESC2012X65N
- U1: footprint WaterNet26 Library:CONV_MIC28514T-E_PHA -> WaterNet Footprints:CONV_MIC28514T-E_PHA
Connections:
- net GND: now also U1.16 (PGND), U1.17 (PGND), U1.18 (PGND), U1.19 (PGND), U1.2 (PGND), U1.22 (PGND), U1.29 (PGND), U1.33 (PGND), U1.33_1 (PGND), U1.33_10 (PGND), U1.33_2 (PGND), U1.33_3 (PGND), U1.33_4 (PGND), U1.33_5 (PGND), U1.33_6 (PGND), U1.33_7 (PGND), U1.33_8 (PGND), U1.33_9 (PGND), U1.36 (PGND), U1.36_1 (PGND), U1.36_2 (PGND), C10.1, C11.1, C12.1, C16.1, C17.1, C18.1, C19.1, J1.1, J1.5, J3.1, J3.5, J4.4, J5.A1 (GND_A), J5.A12 (GND_A), J5.B1 (GND_B), J5.B12 (GND_B), J5.S1 (SHIELD), J5.S2 (SHIELD), J5.S3 (SHIELD), J5.S4 (SHIELD), J7.A1 (GND_A), J7.A12 (GND_A), J7.B1 (GND_B), J7.B12 (GND_B), J7.S1 (SHIELD), J7.S2 (SHIELD), J7.S3 (SHIELD), J7.S4 (SHIELD), R24.1, R25.1, R26.1, R27.1
- net GNDA: now also U1.28 (AGND), R8.1
- net at U1.1 (ILIM): now also R9.1
- net at U1.12 (SW), U1.13 (SW), U1.14 (SW)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: now also C14.2, L1.1, R6.2, R9.2
- net at U1.27 (FB): now also C15.2, C9.1, R7.1, R8.2
- net at U1.4 (BST): now also C14.1
- new net: J5.B5 (CC2), R25.2
- new net: J5.A5 (CC1), R24.2
- new net: C15.1, R6.1
- new net: J7.A5 (CC1), R26.2
- new net: J7.B5 (CC2), R27.2
- new net +5V: C10.2, C11.2, C12.2, C9.2, J1.4, J1.8, J3.4, J3.8, J4.1, L1.2, R7.2
- new net COM_D+: J7.A6 (D1+), J7.B6 (D2+)
- new net COM_D-: J7.A7 (D1-), J7.B7 (D2-)
- new net EXP1_D+: J1.3
- new net EXP1_D-: J1.2
- new net EXP2_D+: J3.3
- new net EXP2_D-: J3.2
- new net JETSON_D+: J4.2, J5.A6 (D1+), J5.B6 (D2+)
- new net JETSON_D-: J4.3, J5.A7 (D1-), J5.B7 (D2-)
- new net PB_D+: J1.7
- new net PB_D-: J1.6
- new net SENS_D+: J3.7
- new net SENS_D-: J3.6
- new net VBUS_A: C16.2, C18.2, J5.A4 (VBUS_A), J5.A9 (VBUS_A), J5.B4 (VBUS_B), J5.B9 (VBUS_B), J7.A4 (VBUS_A), J7.A9 (VBUS_A), J7.B4 (VBUS_B), J7.B9 (VBUS_B), L2.1, L3.1
- new net V_USB_BREAKOUT: C17.2, L2.2
- new net V_USB_COMM: C19.2, L3.2
- no-connect marks 1 -> 3
Other:
- note added: "12V to 5V Regulator"
- note added: "ADAFRUIT Breakout"
- note added: "PORT 1 Sensor Board"
- note added: "PORT 2 Power Board"
- note added: "PORT 3 Exp Board 2"
- note added: "PORT 4 Exp Board 1"
- note added: "USB-C Communication Board (header)"
- note added: "USB-C Jetson"
- moved on the sheet: C1, C2, C3, C4, C5, C6, C7, C8, R1, R2, R3, R4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
