File: boat_pcb_v2/WN_jetson_board/jetson_board.kicad_sch (KiCad schematic)
At the start: 41 parts, among them J1 6130XX11821_61300811821, J3 6130XX11821_61300811821, J4 PPTC041LFBN-RC, J5 USB4120-03-C_REVA6, J6 Conn_02x20_Odd_Even, J7 USB4120-03-C_REVA6, U1 MIC28514T-E_PHA

Commit message: added the remaining headers
Parts:
- added C20, C26: 1µ, 100V, WaterNet Footprints:CAPC2012X145N, symbol Device:C
- added C21, C22: 0.1µ, 25V, WaterNet Footprints:CAPC2012X95N, symbol Device:C
- added C68, C69, C76: 0.1uF 25V, WaterNet Footprints:CAPC2012X95N, symbol WaterNet Library:CL21B104KACNNNC
- added D11: CLMVC-FKA-CL1D1L71BB7C3C3, WaterNet Footprints:LED_CLMVC-FKA-CL1D1L71BB7C3C3, symbol WaterNet Library:CLMVC-FKA-CL1D1L71BB7C3C3
- added J10, J9: Conn_01x12_Pin, symbol Connector:Conn_01x12_Pin
- added JP2, JP3: B04B-PASK-1, WaterNet Footprints:B04B-PASK-1, symbol WaterNet Library:B04B-PASK-1_1
- added R20, R21: 100k, WaterNet Footprints:RES_ERA6AEB104V, symbol Device:R
- added R31, R32, R33: 100 Ohm, WaterNet Footprints:RES_ERJ3EKF1000V, symbol WaterNet Library:ERJ3EKF1000V
- added R66, R67, R68: 10K, WaterNet Footprints:RES_ERA6AEB103V, symbol WaterNet Library:ERA6AEB103V
- added S2, S3: TS04-66-50-BK-160-SMT-TR, WaterNet Footprints:SW_TS04-66-50-BK-160-SMT-TR, symbol WaterNet Library:TS04-66-50-BK-160-SMT-TR
- added U16, U17, U18: BSS123-7-F, WaterNet Footprints:SOT95P240X110-3N, symbol WaterNet Library:BSS123-7-F
- C14, C15: symbol WaterNet26 Library:CL21B104KCFSFNE -> WaterNet Library:CL21B104KCFSFNE
- R24, R25, R26, R27: footprint WaterNet26 Footprints:RESC1508X55N -> WaterNet Footprints:RESC1508X55N; symbol WaterNet26 Library:RMCF0603FT5K10 -> WaterNet Library:RMCF0603FT5K10
Connections:
- net +5V: now also J6.2 (5_VDC), J6.4 (5_VDC)
- net GND: now also J6.14 (GND), J6.20 (GND), J6.25 (GND), J6.34 (GND), J6.39 (GND), J6.6 (GND), J6.9 (GND), C20.2, C21.2, C22.2, C26.2, C68.2, C69.2, C76.2, J9.4 (Pin_4), JP2.1, JP3.1, R66.1, R67.1, R68.1, S2.2, S2.4, S3.2, S3.4, U16.2 (S), U17.2 (S), U18.2 (S)
- net +3.3V: now reaches J6.1 (3.3_VDC)
- net USB_RX: now reaches J6.10 (UART1_RX)
- net USB_RX: now also J10.3 (Pin_3)
- net RGB_B: now reaches J6.15 (GPIO12)
- net RGB_B: now also C68.1, R67.2, U16.1 (G)
- net BUT_1: now reaches J6.29 (GPIO01)
- net BUT_1: now also C21.1, J9.10 (Pin_10), R20.2, S2.1, S2.3
- net I2C1_SDA: now reaches J6.3 (I2C1_SDA)
- net I2C1_SDA: now also J9.1 (Pin_1), JP2.3, JP3.3
- net BUT_2: now reaches J6.31 (GPIO11)
- net BUT_2: now also C22.1, J9.11 (Pin_11), R21.2, S3.1, S3.3
- net RGB_R: now reaches J6.32 (GPIO07)
- net RGB_R: now also C76.1, J10.9 (Pin_9), R68.2, U18.1 (G)
- net I2C1_SCL: now reaches J6.5 (I2C1_SCL)
- net I2C1_SCL: now also J9.2 (Pin_2), JP2.4, JP3.4
- net RGB_G: now reaches J6.7 (GPIO09)
- net RGB_G: now also C69.1, J9.3 (Pin_3), R66.2, U17.1 (G)
- net USB_TX: now reaches J6.8 (UART1_TX)
- net USB_TX: now also J10.2 (Pin_2)
- new net: R31.1, U16.3 (D)
- new net: R33.1, U18.3 (D)
- new net: D11.4, R33.2
- new net: D11.2, R31.2
- new net: R32.1, U17.3 (D)
- new net: D11.3, R32.2
- new net +3V3: C20.1, C26.1, D11.1, JP2.2, JP3.2, R20.1, R21.1
- new net GPIO12: J9.7 (Pin_7)
- new net GPIO13: J9.12 (Pin_12)
- new net I2C0_SCK: J9.9 (Pin_9)
- new net I2C0_SCL: J10.8 (Pin_8)
- new net I2S0_FS: J10.1 (Pin_1)
- new net I2S0_SCLK: J10.4 (Pin_4)
- new net I2S0_SDIN: J10.11 (Pin_11)
- new net I2S0_SDOUT: J10.12 (Pin_12)
- new net SP11_SCK: J9.6 (Pin_6)
- new net SPI0_CS1: J10.7 (Pin_7)
- new net SPI0_MISO: J9.8 (Pin_8)
- new net SPI1_CS1: J10.5 (Pin_5)
- new net SPI1_MISO: J10.6 (Pin_6)
- new net UART1_RTS: J9.5 (Pin_5)
- new net UART_CTS: J10.10 (Pin_10)
Other:
- note added: "Button 1"
- note added: "Button 2"
- note added: "HEADER"
- note added: "I2C QWIIC CONN"
- note added: "JETSON BREAKOUT HEADER"
- note added: "Onboard RGB LED"
- moved on the sheet: J1, J3, J4, J6

Commit message: minor updates related to board layout
Connections:
- net +12V renamed +VBAT
Changed lines of the file:
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@@
 		(on_board yes)
 		(dnp no)
-		(fields_autoplaced yes)
 		(property "Reference" "#PWR01"
 			(at 38.1 74.93 0)
@@
 			)
 		)
-		(property "Value" "+12V"
-			(at 38.1 66.04 0)
+		(property "Value" "+VBAT"
+			(at 35.56 66.548 0)
 			(effects
 				(font
 					(size 1.27 1.27)
 				)
+				(justify left)
 			)
 		)

Commit message: Changed the Regulator on Jetson to Vbat to 12V
Parts:
- removed R8: 1.37k 0.5%, WaterNet Footprints:RESC1608X55N, symbol WaterNet Library:RT0603DRD071K37L
- removed R9: 1.42k, WaterNet Footprints:RESC1608X55N, symbol WaterNet Library:RT0603BRD071K42L
- added R28: 1.5K 1%, WaterNet Footprints:RES_ERJ3EKF1501V, symbol WaterNet26 Library:ERJ3EKF1501V
- added R29: ERA-3AEB4990V, WaterNet Footprints:RESC1608X55N, symbol WaterNet26 Library:ERA-3AEB4990V
Connections:
- net +5V: no longer C10.2, C11.2, C12.2, C9.2, L1.2, R7.2
- net GNDA: now also R29.1
- net at C15.2, C9.1, R7.1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: now also R29.2
- net at U1.1 (ILIM): now also R28.1
- net at C14.2, L1.1, R6.2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: now also R28.2
- new net +12V: C10.2, C11.2, C12.2, C9.2, L1.2, R7.2
Other:
- note added: "VBAT to 12V Regulator"
- note removed: "12V to 5V Regulator"
